Commit message: feat(robot_description): consume independent sensor facts

File: core/robot/robot_description/gazebo/robot.gazebo.xacro (robot description, xacro)
@@ -2,5 +2,5 @@
 <robot xmlns:xacro="http://www.ros.org/wiki/xacro">
   <!-- prefix: link 名前缀(与本体宏一致)；gz_controllers_file: gz_ros2_control 读取的控制器 yaml 绝对路径，由 launch 注入 -->
-  <xacro:macro name="robot_gazebo" params="prefix gz_controllers_file">
+  <xacro:macro name="robot_gazebo" params="prefix gz_controllers_file lidar_scan_lines lidar_columns_per_scan lidar_scan_rate_hz lidar_min_range lidar_max_range lidar_horizontal_start_angle lidar_horizontal_end_angle imu_rate_hz">
     <!-- gz_ros2_control：controller_manager 随 Gz 进程起 -->
     <gazebo>
@@ -20,11 +20,10 @@
       <preserveFixedJoint>true</preserveFixedJoint>
     </gazebo>
-    <!-- 雷达：Gz 原生 gpu_lidar，16 线 / ±15° / 1800 水平(对齐 N_SCAN=16、Horizon_SCAN=1800)。
-         参数取自已验证的 Phase 0 spike。显式 topic=lidar(点云在 lidar/points)，避免 spawn 模型作用域前缀。 -->
+    <!-- 雷达：Gz 原生 gpu_lidar。显式 topic=lidar(点云在 lidar/points)，避免 spawn 模型作用域前缀。 -->
     <gazebo reference="${prefix}velodyne">
       <sensor name="gpu_lidar" type="gpu_lidar">
         <topic>lidar</topic>
         <gz_frame_id>${prefix}velodyne</gz_frame_id>
-        <update_rate>10</update_rate>
+        <update_rate>${lidar_scan_rate_hz}</update_rate>
         <always_on>1</always_on>
         <visualize>true</visualize>
@@ -32,11 +31,11 @@
           <scan>
             <horizontal>
-              <samples>1800</samples>
+              <samples>${lidar_columns_per_scan}</samples>
               <resolution>1</resolution>
-              <min_angle>-3.14159</min_angle>
-              <max_angle>3.14159</max_angle>
+              <min_angle>${lidar_horizontal_start_angle}</min_angle>
+              <max_angle>${lidar_horizontal_end_angle}</max_angle>
             </horizontal>
             <vertical>
-              <samples>16</samples>
+              <samples>${lidar_scan_lines}</samples>
               <resolution>1</resolution>
               <min_angle>-0.261799</min_angle>
@@ -45,6 +44,6 @@
           </scan>
           <range>
-            <min>0.9</min>
-            <max>100.0</max>
+            <min>${lidar_min_range}</min>
+            <max>${lidar_max_range}</max>
             <resolution>0.01</resolution>
           </range>
@@ -52,10 +51,10 @@
       </sensor>
     </gazebo>
-    <!-- IMU：Gz 原生 imu，与 velodyne 共位。显式 topic=imu。 -->
+    <!-- IMU：Gz 原生 imu。显式 topic=imu。 -->
     <gazebo reference="${prefix}imu_link">
       <sensor name="imu" type="imu">
         <topic>imu</topic>
         <gz_frame_id>${prefix}imu_link</gz_frame_id>
-        <update_rate>200</update_rate>
+        <update_rate>${imu_rate_hz}</update_rate>
         <always_on>1</always_on>
       </sensor>

File: core/robot/robot_description/urdf/robot.urdf.xacro (robot description, xacro)
@@ -13,10 +13,24 @@
   <xacro:arg name="wheel_width" default="0.06"/>
   <xacro:arg name="wheel_separation" default="0.55"/>
-  <xacro:arg name="sensor_x" default="0.0"/>
-  <xacro:arg name="sensor_y" default="0.0"/>
-  <xacro:arg name="sensor_z" default="0.236"/>
-  <xacro:arg name="sensor_roll" default="0.0"/>
-  <xacro:arg name="sensor_pitch" default="0.0"/>
-  <xacro:arg name="sensor_yaw" default="0.0"/>
+  <xacro:arg name="lidar_x" default="0.0"/>
+  <xacro:arg name="lidar_y" default="0.0"/>
+  <xacro:arg name="lidar_z" default="0.236"/>
+  <xacro:arg name="lidar_roll" default="0.0"/>
+  <xacro:arg name="lidar_pitch" default="0.0"/>
+  <xacro:arg name="lidar_yaw" default="0.0"/>
+  <xacro:arg name="imu_x" default="0.0"/>
+  <xacro:arg name="imu_y" default="0.0"/>
+  <xacro:arg name="imu_z" default="0.236"/>
+  <xacro:arg name="imu_roll" default="0.0"/>
+  <xacro:arg name="imu_pitch" default="0.0"/>
+  <xacro:arg name="imu_yaw" default="0.0"/>
+  <xacro:arg name="lidar_scan_lines" default="16"/>
+  <xacro:arg name="lidar_columns_per_scan" default="1800"/>
+  <xacro:arg name="lidar_scan_rate_hz" default="10"/>
+  <xacro:arg name="lidar_min_range" default="0.9"/>
+  <xacro:arg name="lidar_max_range" default="100.0"/>
+  <xacro:arg name="lidar_horizontal_start_angle" default="-3.14159"/>
+  <xacro:arg name="lidar_horizontal_end_angle" default="3.14159"/>
+  <xacro:arg name="imu_rate_hz" default="200"/>
   <!-- 仅 Gz 模式用：gz_ros2_control 读取的控制器 yaml 绝对路径 -->
   <xacro:arg name="gz_controllers_file" default=""/>
@@ -33,5 +47,15 @@
   <xacro:if value="$(arg use_gazebo)">
     <xacro:include filename="$(find robot_description)/gazebo/robot.gazebo.xacro"/>
-    <xacro:robot_gazebo prefix="$(arg prefix)" gz_controllers_file="$(arg gz_controllers_file)"/>
+    <xacro:robot_gazebo
+      prefix="$(arg prefix)"
+      gz_controllers_file="$(arg gz_controllers_file)"
+      lidar_scan_lines="$(arg lidar_scan_lines)"
+      lidar_columns_per_scan="$(arg lidar_columns_per_scan)"
+      lidar_scan_rate_hz="$(arg lidar_scan_rate_hz)"
+      lidar_min_range="$(arg lidar_min_range)"
+      lidar_max_range="$(arg lidar_max_range)"
+      lidar_horizontal_start_angle="$(arg lidar_horizontal_start_angle)"
+      lidar_horizontal_end_angle="$(arg lidar_horizontal_end_angle)"
+      imu_rate_hz="$(arg imu_rate_hz)"/>
   </xacro:if>
 </robot>

File: core/robot/robot_description/urdf/robot_macro.urdf.xacro (robot description, xacro)
@@ -1,5 +1,5 @@
 <?xml version="1.0"?>
 <!-- 差速移动底盘本体(默认参数为仿真尺寸，真机由 system_bringup 覆盖；根=base_footprint(REP-105 地面投影帧)，其下 base_link 为车体)：盒身 + 左右驱动轮
-     + 前后球形万向轮(半径=驱动轮、同高) + 车顶中央共位的 velodyne / imu_link 挂载帧。
+     + 前后球形万向轮(半径=驱动轮、同高) + 独立的 velodyne / imu_link 挂载帧。
      碰撞用基本几何(box/cylinder/sphere)。Gz 传感器插件在 Phase 3 的 gazebo.xacro 加。
      注：base_footprint 无 inertial 作根，base_link(带 inertial)为其固定子，
@@ -30,10 +30,16 @@
   <xacro:property name="wheel_z"  value="${wheel_radius - base_link_height}"/>
   <xacro:property name="caster_x" value="${base_length/2 - caster_radius}"/>
-  <xacro:property name="sensor_x" value="$(arg sensor_x)"/>
-  <xacro:property name="sensor_y" value="$(arg sensor_y)"/>
-  <xacro:property name="sensor_z" value="$(arg sensor_z)"/>
-  <xacro:property name="sensor_roll" value="$(arg sensor_roll)"/>
-  <xacro:property name="sensor_pitch" value="$(arg sensor_pitch)"/>
-  <xacro:property name="sensor_yaw" value="$(arg sensor_yaw)"/>
+  <xacro:property name="lidar_x" value="$(arg lidar_x)"/>
+  <xacro:property name="lidar_y" value="$(arg lidar_y)"/>
+  <xacro:property name="lidar_z" value="$(arg lidar_z)"/>
+  <xacro:property name="lidar_roll" value="$(arg lidar_roll)"/>
+  <xacro:property name="lidar_pitch" value="$(arg lidar_pitch)"/>
+  <xacro:property name="lidar_yaw" value="$(arg lidar_yaw)"/>
+  <xacro:property name="imu_x" value="$(arg imu_x)"/>
+  <xacro:property name="imu_y" value="$(arg imu_y)"/>
+  <xacro:property name="imu_z" value="$(arg imu_z)"/>
+  <xacro:property name="imu_roll" value="$(arg imu_roll)"/>
+  <xacro:property name="imu_pitch" value="$(arg imu_pitch)"/>
+  <xacro:property name="imu_yaw" value="$(arg imu_yaw)"/>
   <!-- base_footprint：REP-105 地面投影根帧(无质量)。LIO-SAM baselinkFrame / Nav2 用。 -->
   <link name="${prefix}base_footprint"/>
@@ -169,9 +175,9 @@
     </inertial>
   </link>
-  <!-- 雷达挂载帧 velodyne：车顶中央、puck 底贴车顶、完全外露。Phase 3 在此挂 Gz gpu_lidar。 -->
+  <!-- 雷达挂载帧 velodyne：Phase 3 在此挂 Gz gpu_lidar。 -->
   <joint name="${prefix}velodyne_joint" type="fixed">
     <parent link="${prefix}base_link"/>
     <child  link="${prefix}velodyne"/>
-    <origin xyz="${sensor_x} ${sensor_y} ${sensor_z}" rpy="${sensor_roll} ${sensor_pitch} ${sensor_yaw}"/>
+    <origin xyz="${lidar_x} ${lidar_y} ${lidar_z}" rpy="${lidar_roll} ${lidar_pitch} ${lidar_yaw}"/>
   </joint>
   <link name="${prefix}velodyne">
@@ -194,9 +200,9 @@
     </inertial>
   </link>
-  <!-- IMU 挂载帧 imu_link：与 velodyne 同位置(外参归零)。Phase 3 在此挂 Gz imu。 -->
+  <!-- IMU 挂载帧 imu_link：Phase 3 在此挂 Gz imu。 -->
   <joint name="${prefix}imu_joint" type="fixed">
     <parent link="${prefix}base_link"/>
     <child  link="${prefix}imu_link"/>
-    <origin xyz="${sensor_x} ${sensor_y} ${sensor_z}" rpy="${sensor_roll} ${sensor_pitch} ${sensor_yaw}"/>
+    <origin xyz="${imu_x} ${imu_y} ${imu_z}" rpy="${imu_roll} ${imu_pitch} ${imu_yaw}"/>
   </joint>
   <link name="${prefix}imu_link">
